File: kicad/ad8066_filter/ad8066_filter.kicad_pcb (KiCad board)
At the start: 2 copper layers, 25.4 x 25.4 mm, 18 parts, among them J1 Conn_01x03, J2 Conn_01x03, U1 AD8066

Commit message: updated
Parts:
- moved R8 0.13 mm to (171.7, 95.5)
- moved C6 0.13 mm to (172.7, 88.0)
Routing:
- net /5V: track 27.6 -> 30.2 mm
- net /GND: track 8.26 -> 10.4 mm
Other:
- board text added: "5V"
- board text added: "GND"
- board text added: "IF"
- board text added: "OUT1"
- board text added: "OUT2"
- board text added: "ad8066_filter iman_202001.1"
- board text removed: "ad8066_filter iman_20191230"
Changed lines of the file:
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@@
-(kicad_pcb (version 20171130) (host pcbnew "(5.1.5)-3")
+(kicad_pcb (version 20171130) (host pcbnew "(5.1.5)-2")
   (general
     (thickness 1.6)
-    (drawings 8)
-    (tracks 92)
+    (drawings 14)
+    (tracks 96)
     (zones 0)
     (modules 18)
@@
   )
   (page A4)
+  (title_block
+    (title "AD8066 Filter board")
+    (date 2019-12-31)
+    (rev 1)
+    (company Iman)
+  )
   (layers
     (0 F.Cu signal)
@@
     (43 Eco2.User user hide)
     (44 Edge.Cuts user)
-    (45 Margin user hide)
+    (45 Margin user)
     (46 B.CrtYd user hide)
     (47 F.CrtYd user hide)
@@
       (drillshape 0)
       (scaleselection 1)
-      (outputdirectory "releases/ad8066-filter_20191230"))
+      (outputdirectory "releases/ad8066-filter_20200101"))
   )
   (net 0 "")
@@
   )
   (module Resistor_SMD:R_0805_2012Metric_Pad1.15x1.40mm_HandSolder (layer F.Cu)
-    (at 171.831 95.495 90)
+    (at 171.704 95.504 90)
     (descr "Resistor SMD 0805 (2012 Metric), square (rectangular) end terminal, IPC_7351 nominal with elongated pad for handsoldering. (Body size source: https://docs.google.com/spreadsheets/d/1BsfQQcO9C6DZCsRaXUlFlo91Tg2WpOkGARC1WS5S8t0/edit?usp=sharing), generated with kicad-footprint-generator")
     (tags "resistor handsolder")
@@
   )
   (module LED_SMD:LED_0805_2012Metric_Pad1.15x1.40mm_HandSolder (layer F.Cu)
-    (at 173.99 95.513 90)
+    (at 173.99 95.504 90)
     (descr "LED SMD 0805 (2012 Metric), square (rectangular) end terminal, IPC_7351 nominal, (Body size source: https://docs.google.com/spreadsheets/d/1BsfQQcO9C6DZCsRaXUlFlo91Tg2WpOkGARC1WS5S8t0/edit?usp=sharing), generated with kicad-footprint-generator")
     (tags "LED handsolder")
@@
   )
   (module Capacitor_SMD:C_0805_2012Metric_Pad1.15x1.40mm_HandSolder (layer F.Cu)
-    (at 172.847 88.011)
+    (at 172.72 88.011)
     (descr "Capacitor SMD 0805 (2012 Metric), square (rectangular) end terminal, IPC_7351 nominal with elongated pad for handsoldering. (Body size source: https://docs.google.com/spreadsheets/d/1BsfQQcO9C6DZCsRaXUlFlo91Tg2WpOkGARC1WS5S8t0/edit?usp=sharing), generated with kicad-footprint-generator")
     (tags "capacitor handsolder")
@@
     (descr "Through hole straight pin header, 1x03, 2.54mm pitch, single row")
     (tags "Through hole pin header THT 1x03 2.54mm single row")
-    (fp_text reference J1 (at 1.905 6.096) (layer F.SilkS)
+    (fp_text reference J1 (at 1.016 7.239) (layer F.SilkS)
       (effects (font (size 0.508 0.508) (thickness 0.0762)))
     )
@@
     )
   )
-  (gr_text "ad8066_filter\niman_20191230" (at 173.101 78.486) (layer F.SilkS)
+  (gr_text 5V (at 162.56 98.679) (layer F.SilkS)
+    (effects (font (size 0.381 0.381) (thickness 0.0762)))
+  )
+  (gr_text IF (at 165.1 98.679) (layer F.SilkS)
+    (effects (font (size 0.381 0.381) (thickness 0.0762)))
+  )
+  (gr_text GND (at 167.64 98.679) (layer F.SilkS)
+    (effects (font (size 0.381 0.381) (thickness 0.0762)))
+  )
+  (gr_text OUT1 (at 162.56 79.375) (layer F.SilkS)
+    (effects (font (size 0.381 0.381) (thickness 0.0762)))
+  )
+  (gr_text OUT2 (at 167.64 79.375) (layer F.SilkS)
+    (effects (font (size 0.381 0.381) (thickness 0.0762)))
+  )
+  (gr_text GND (at 165.1 79.375) (layer F.SilkS)
+    (effects (font (size 0.381 0.381) (thickness 0.0762)))
+  )
+  (gr_text "ad8066_filter\niman_202001.1" (at 173.101 78.486) (layer F.SilkS)
     (effects (font (size 0.508 0.508) (thickness 0.0762)))
   )
@@
   (gr_line (start 177.8 101.6) (end 177.8 76.2) (layer Edge.Cuts) (width 0.05))
   (gr_line (start 152.4 101.6) (end 177.8 101.6) (layer Edge.Cuts) (width 0.05))
-  (via (at 168.783 88.011) (size 0.8) (drill 0.4) (layers F.Cu B.Cu) (net 10))
-  (via (at 173.863 88.011) (size 0.8) (drill 0.4) (layers F.Cu B.Cu) (net 8))
   (segment (start 158.01399 89.92399) (end 158.006 89.916) (width 0.254) (layer F.Cu) (net 1))
   (segment (start 156.972 90.375) (end 157.431 89.916) (width 0.254) (layer F.Cu) (net 1))
@@
   (segment (start 165.989 83.82) (end 167.876 83.82) (width 0.254) (layer F.Cu) (net 6))
   (segment (start 167.876 84.973933) (end 167.876 83.82) (width 0.254) (layer F.Cu) (net 6))
-  (segment (start 167.386 86.552943) (end 167.876 86.062943) (width 0.254) (layer F.Cu) (net 6))
-  (segment (start 167.386 90.050067) (end 167.386 86.552943) (width 0.254) (layer F.Cu) (net 6))
-  (segment (start 167.876 86.062943) (end 167.876 83.82) (width 0.254) (layer F.Cu) (net 6))
+  (segment (start 167.386 90.050067) (end 167.386 85.707) (width 0.254) (layer F.Cu) (net 6))
+  (segment (start 167.386 85.707) (end 167.876 85.217) (width 0.254) (layer F.Cu) (net 6))
   (segment (start 168.7 90.551) (end 167.886933 90.551) (width 0.254) (layer F.Cu) (net 6))
   (segment (start 167.886933 90.551) (end 167.386 90.050067) (width 0.254) (layer F.Cu) (net 6))
+  (segment (start 167.876 85.217) (end 167.876 83.82) (width 0.254) (layer F.Cu) (net 6))
   (segment (start 169.926 81.679) (end 169.944 81.661) (width 0.254) (layer F.Cu) (net 7))
   (segment (start 169.926 83.82) (end 169.926 81.679) (width 0.254) (layer F.Cu) (net 7))
@@
   (segment (start 169.5 89.281) (end 169.926 88.855) (width 0.254) (layer F.Cu) (net 7))
   (segment (start 168.7 89.281) (end 169.5 89.281) (width 0.254) (layer F.Cu) (net 7))
-  (segment (start 173.99 97.113) (end 173.99 96.538) (width 0.254) (layer F.Cu) (net 8))
-  (segment (start 170.773 100.33) (end 173.99 97.113) (width 0.254) (layer F.Cu) (net 8))
-  (segment (start 167.64 100.33) (end 170.773 100.33) (width 0.254) (layer F.Cu) (net 8))
+  (via (at 173.863 88.011) (size 0.8) (drill 0.4) (layers F.Cu B.Cu) (net 8))
   (segment (start 157.988 95.123) (end 157.988 95.123) (width 0.254) (layer F.Cu) (net 8))
   (segment (start 161.5 91.821) (end 161.5 91.821) (width 0.254) (layer F.Cu) (net 8))
@@
   (via (at 157.988 95.123) (size 0.8) (drill 0.4) (layers F.Cu B.Cu) (net 8))
   (segment (start 173.99 96.538) (end 173.99 96.538) (width 0.254) (layer F.Cu) (net 8))
-  (via (at 173.99 96.538) (size 0.8) (drill 0.4) (layers F.Cu B.Cu) (net 8))
-  (via (at 161.5 91.821) (size 0.8) (drill 0.4) (layers F.Cu B.Cu) (net 8))
+  (via (at 159.639 92.456) (size 0.8) (drill 0.4) (layers F.Cu B.Cu) (net 8))
+  (segment (start 173.99 97.104) (end 173.99 96.529) (width 0.25) (layer F.Cu) (net 8))
+  (segment (start 170.764 100.33) (end 173.99 97.104) (width 0.25) (layer F.Cu) (net 8))
+  (segment (start 167.64 100.33) (end 170.764 100.33) (width 0.25) (layer F.Cu) (net 8))
+  (segment (start 173.99 96.529) (end 173.99 96.529) (width 0.25) (layer F.Cu) (net 8))
+  (via (at 173.99 96.529) (size 0.8) (drill 0.4) (layers F.Cu B.Cu) (net 8))
+  (segment (start 160.274 91.821) (end 159.639 92.456) (width 0.254) (layer F.Cu) (net 8))
+  (segment (start 161.5 91.821) (end 160.274 91.821) (width 0.254) (layer F.Cu) (net 8))
   (segment (start 155.938 99.187) (end 155.974 99.187) (width 0.254) (layer F.Cu) (net 9))
   (segment (start 155.938 95.123) (end 155.938 97.155) (width 0.254) (layer F.Cu) (net 9))
@@
   (segment (start 155.938 94.423) (end 155.938 92.075) (width 0.254) (layer F.Cu) (net 9))
   (segment (start 155.938 95.123) (end 155.938 94.423) (width 0.254) (layer F.Cu) (net 9))
+  (via (at 168.91 85.979) (size 0.8) (drill 0.4) (layers F.Cu B.Cu) (net 10))
   (segment (start 171.831 88.02) (end 171.822 88.011) (width 0.254) (layer F.Cu) (net 10))
   (segment (start 171.831 94.47) (end 171.831 94.47) (width 0.254) (layer F.Cu) (net 10))
@@
   (segment (start 158.431 100.33) (end 157.988 99.887) (width 0.254) (layer F.Cu) (net 10))
   (segment (start 162.56 100.33) (end 158.431 100.33) (width 0.254) (layer F.Cu) (net 10))
-  (via (at 171.831 94.47) (size 0.8) (drill 0.4) (layers F.Cu B.Cu) (net 10))
-  (segment (start 166.808 94.47) (end 171.131 94.47) (width 0.762) (layer B.Cu) (net 10))
-  (segment (start 171.131 94.47) (end 171.831 94.47) (width 0.762) (layer B.Cu) (net 10))
-  (segment (start 162.56 98.718) (end 166.808 94.47) (width 0.762) (layer B.Cu) (net 10))
+  (via (at 171.704 94.47) (size 0.8) (drill 0.4) (layers F.Cu B.Cu) (net 10))
   (segment (start 162.56 100.33) (end 162.56 98.718) (width 0.762) (layer B.Cu) (net 10))
   (segment (start 171.822 88.011) (end 171.822 88.011) (width 0.254) (layer F.Cu) (net 10))
-  (via (at 171.822 88.011) (size 0.8) (drill 0.4) (layers F.Cu B.Cu) (net 10))
-  (segment (start 171.831 88.02) (end 171.822 88.011) (width 0.762) (layer B.Cu) (net 10))
-  (segment (start 171.831 94.47) (end 171.831 88.02) (width 0.762) (layer B.Cu) (net 10))
-  (segment (start 171.822 88.011) (end 168.783 88.011) (width 0.762) (layer B.Cu) (net 10))
+  (via (at 171.704 88.011) (size 0.8) (drill 0.4) (layers F.Cu B.Cu) (net 10))
+  (segment (start 171.704 94.488) (end 171.704 88.038) (width 0.762) (layer B.Cu) (net 10))
+  (segment (start 166.808 94.47) (end 162.56 98.718) (width 0.762) (layer B.Cu) (net 10))
+  (segment (start 171.704 94.47) (end 166.808 94.47) (width 0.762) (layer B.Cu) (net 10))
+  (segment (start 168.7 86.189) (end 168.91 85.979) (width 0.762) (layer F.Cu) (net 10))
+  (segment (start 168.7 88.011) (end 168.7 86.189) (width 0.762) (layer F.Cu) (net 10))
+  (segment (start 169.672 85.979) (end 171.704 88.011) (width 0.762) (layer B.Cu) (net 10))
+  (segment (start 168.91 85.979) (end 169.672 85.979) (width 0.762) (layer B.Cu) (net 10))
   (segment (start 161.5 90.551) (end 161.5 90.551) (width 0.254) (layer F.Cu) (net 11))
   (segment (start 160.7 90.551) (end 161.5 90.551) (width 0.254) (layer F.Cu) (net 11))
